File: kicad8/kicad8.kicad_pcb (KiCad board)
At the start: 2 copper layers, 314.5 x 124 mm, 192 parts, among them J1 USB_C_Receptacle_USB2.0, SW1 RotaryEncoder_Switch, U1 STM32F072CBT6, U2 PRTR5V0U2X, U3 XC6206PxxxMR-Regulator_Linear

Commit message: -Added: Ground fill
Parts:
- moved BOOT1 148.8 mm to (305.6, 83.6), turned to 90 degrees
- moved R3 141.7 mm to (303.6, 77.5), turned to 180 degrees
- moved RST1 141.1 mm to (299.3, 83.6), turned to 90 degrees
- moved R4 138.5 mm to (301.1, 77.5), turned to 180 degrees
- moved C1 136.6 mm to (300.8, 75.3), turned to 180 degrees
- moved C6 19.2 mm to (309.3, 63.8)
- moved C7 19.2 mm to (305.9, 68.3)
- moved C5 19.2 mm to (308.5, 62.4)
- moved U1 19.2 mm to (302.3, 62.5)
- moved C2 19.2 mm to (300.9, 53.4)
- moved C3 19.2 mm to (302.1, 56.4)
- moved C4 19.2 mm to (295.9, 62.6)
- moved C8 0.27 mm to (305.1, 28.8)
- moved F1 0.27 mm to (302.1, 29.6)
- moved J1 0.27 mm to (302.2, 17.5)
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Connections:
- U1 pad 10: /A0 -> col13
- U1 pad 11: /A1 -> col11
- U1 pad 12: /A2 -> col10
- U1 pad 13: /A3 -> col9
- U1 pad 14: col14 -> col8
- U1 pad 15: col13 -> col7
- U1 pad 16: col12 -> col6
- U1 pad 17: col11 -> col5
- U1 pad 18: col10 -> col4
- U1 pad 19: col9 -> col3
- U1 pad 2: rot1 -> /C13
- U1 pad 20: col8 -> col2
- U1 pad 21: col7 -> col1
- U1 pad 22: /B11 -> col0
- U1 pad 25: col6 -> col12
- U1 pad 26: col5 -> /B13
- U1 pad 27: col4 -> /B14
- U1 pad 28: col3 -> /B15
- U1 pad 29: col2 -> /A8
- U1 pad 3: rot0 -> row2
- U1 pad 30: col1 -> /A9
- U1 pad 31: col0 -> /A10
- U1 pad 37: row2 -> row0
- U1 pad 38: row1 -> rot1
- U1 pad 39: row0 -> rot0
- U1 pad 4: /C15 -> row3
- U1 pad 40: /B4 -> row1
- U1 pad 41: row5 -> /B5
- U1 pad 42: row4 -> /B6
- U1 pad 43: row3 -> col14
- U1 pad 5: /F0 -> row4
- U1 pad 6: /F1 -> row5
Routing:
- net GND: track 371.1 -> 166.0 mm, vias 8 -> 6
- net +3V3: track 281.2 -> 98.6 mm, vias 6 -> 5
- net BOOT0: track 202.4 -> 31.9 mm, vias 6 -> 2
- net NRST: track 189.4 -> 27.7 mm, vias 4 -> 2
- net col3: track 374.3 -> 307.5 mm
- net row0: track 378.9 -> 328.7 mm
- net row1: track 343.4 -> 306.1 mm, vias 0 -> 2
- net rot0: track 71.6 -> 41.1 mm, vias 1 -> 0
- net rot1: track 62.4 -> 35.6 mm, vias 1 -> 0
- net col14: track 143.0 -> 119.7 mm
- net D+: track 63.5 -> 43.2 mm, vias 2 -> 0
- net D-: track 61.7 -> 42.1 mm, vias 2 -> 0
- net row4: track 360.0 -> 345.3 mm, vias 0 -> 2
- net col13: track 143.8 -> 156.3 mm
- net row5: track 372.7 -> 361.6 mm
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- added copper zone on B.Cu, net GND
- added copper zone on F.Cu, net GND
